File: hotline/display.kicad_sch (KiCad schematic)
At the start: 17 parts, among them Q1 2N7002H, Q2 2N7002H, Q3 2N7002H, Q4 2N7002H, Q5 2N7002H, Q6 2N7002H, Q7 2N7002H, Q8 2N7002H

Commit message: assign footprints
Signed-off-by: Kolbjørn Austreng <kolbjorn.austreng@example.com>
Parts:
- J3: renamed from J; footprint (none) -> Connector_Molex:Molex_PicoBlade_53261-1071_1x10-1MP_P1.25mm_Horizontal
- R23: renamed from R21; footprint (none) -> Resistor_SMD:R_0603_1608Metric_Pad0.98x0.95mm_HandSolder
- R24: renamed from R22; footprint (none) -> Resistor_SMD:R_0603_1608Metric_Pad0.98x0.95mm_HandSolder
- R25: renamed from R23; footprint (none) -> Resistor_SMD:R_0603_1608Metric_Pad0.98x0.95mm_HandSolder
- R26: renamed from R24; footprint (none) -> Resistor_SMD:R_0603_1608Metric_Pad0.98x0.95mm_HandSolder
- R27: renamed from R20; footprint (none) -> Resistor_SMD:R_0603_1608Metric_Pad0.98x0.95mm_HandSolder
- R28: renamed from R18; footprint (none) -> Resistor_SMD:R_0603_1608Metric_Pad0.98x0.95mm_HandSolder
- R29: renamed from R19; footprint (none) -> Resistor_SMD:R_0603_1608Metric_Pad0.98x0.95mm_HandSolder
- R30: renamed from R17; footprint (none) -> Resistor_SMD:R_0603_1608Metric_Pad0.98x0.95mm_HandSolder
- renumbered Q5 to Q1, Q6 to Q2, Q7 to Q3, Q8 to Q4, Q4 to Q5, Q2 to Q6, Q3 to Q7, Q1 to Q8
