File: hotline/audio_out.kicad_sch (KiCad schematic)
At the start: 31 parts, among them U3 NC7WZ16, U4 LM4040DBZ-2.5, U5 TDA2822D

Commit message: assign footprints
Signed-off-by: Kolbjørn Austreng <kolbjorn.austreng@example.com>
Parts:
- C11: renamed from C18; footprint (none) -> Capacitor_SMD:CP_Elec_4x5.7
- C12: renamed from C19; footprint (none) -> Capacitor_SMD:C_0603_1608Metric_Pad1.08x0.95mm_HandSolder
- C13: renamed from C17; footprint (none) -> Capacitor_SMD:CP_Elec_5x5.3
- C14: renamed from C10; footprint (none) -> Capacitor_SMD:C_0603_1608Metric_Pad1.08x0.95mm_HandSolder
- C15: renamed from C11; footprint (none) -> Capacitor_SMD:C_0805_2012Metric_Pad1.18x1.45mm_HandSolder
- C16: renamed from C12; footprint (none) -> Capacitor_SMD:C_0603_1608Metric_Pad1.08x0.95mm_HandSolder
- C17: renamed from C13; footprint (none) -> Capacitor_SMD:CP_Elec_4x5.7
- C18: renamed from C16; footprint (none) -> Capacitor_SMD:CP_Elec_8x10
- C19: renamed from C15; footprint (none) -> Capacitor_SMD:C_0603_1608Metric_Pad1.08x0.95mm_HandSolder
- C20: renamed from C14; footprint (none) -> Capacitor_SMD:C_0603_1608Metric_Pad1.08x0.95mm_HandSolder
- C21: renamed from C8; footprint (none) -> Capacitor_SMD:C_0603_1608Metric_Pad1.08x0.95mm_HandSolder
- C22: renamed from C9; footprint (none) -> Capacitor_SMD:C_0805_2012Metric_Pad1.18x1.45mm_HandSolder
- JP1, JP3: footprint (none) -> Jumper:SolderJumper-2_P1.3mm_Bridged_RoundedPad1.0x1.5mm
- JP2, JP4: footprint (none) -> Jumper:SolderJumper-2_P1.3mm_Open_RoundedPad1.0x1.5mm
- LS1: footprint (none) -> TerminalBlock_Phoenix:TerminalBlock_Phoenix_PT-1,5-2-5.0-H_1x02_P5.00mm_Horizontal
- R14: renamed from R10; footprint (none) -> Resistor_SMD:R_0603_1608Metric_Pad0.98x0.95mm_HandSolder
- R15: renamed from R12; footprint (none) -> Resistor_SMD:R_0603_1608Metric_Pad0.98x0.95mm_HandSolder
- R16: value R_Small -> 10k; footprint (none) -> Resistor_SMD:R_0603_1608Metric_Pad0.98x0.95mm_HandSolder
- R17: renamed from R13; footprint (none) -> Resistor_SMD:R_0603_1608Metric_Pad0.98x0.95mm_HandSolder
- R18: renamed from R11; footprint (none) -> Resistor_SMD:R_0603_1608Metric_Pad0.98x0.95mm_HandSolder
- R19: renamed from R15; footprint (none) -> Resistor_SMD:R_0603_1608Metric_Pad0.98x0.95mm_HandSolder
- R20: renamed from R14; footprint (none) -> Resistor_SMD:R_0603_1608Metric_Pad0.98x0.95mm_HandSolder
- R21: renamed from R8; footprint (none) -> Resistor_SMD:R_0603_1608Metric_Pad0.98x0.95mm_HandSolder
- R22: renamed from R9; footprint (none) -> Resistor_SMD:R_0603_1608Metric_Pad0.98x0.95mm_HandSolder
- U3: footprint (none) -> Package_TO_SOT_SMD:SOT-363_SC-70-6_Handsoldering
- U5: footprint (none) -> Package_SO:SOIC-8_3.9x4.9mm_P1.27mm
- renumbered D2 to D3, D1 to D4

Commit message: place components
Signed-off-by: Kolbjørn Austreng <kolbjorn.austreng@example.com>
Parts:
- added JP5: Bridged, Jumper:SolderJumper-2_P1.3mm_Bridged_RoundedPad1.0x1.5mm, symbol Jumper:SolderJumper_2_Bridged
- added R40, R41, R42, R43: 100, Resistor_SMD:R_0603_1608Metric_Pad0.98x0.95mm_HandSolder, symbol Device:R_Small
Connections:
- net +3V3: now also R40.2, R41.2, R42.2, R43.2; no longer U3.5 (V_{CC}), U4.1 (K)
- net at R19.1, U5.3 (Out2): now also JP5.2 (B); no longer JP4.2 (B), LS1.2
- new net: R40.1, R41.1, R42.1, R43.1, U3.5 (V_{CC}), U4.1 (K)
- new net: JP4.2 (B), JP5.1 (A), LS1.2
Other:
- moved on the sheet: C14, C15, C19, D3, R14, R15, R17, R18, R19, U3, U4
