File: hotline/hotline.kicad_pcb (KiCad board)
At the start: 4 copper layers, 100 x 74.5 mm, 107 parts, among them J1 USB_C_Receptacle_PowerOnly_24P, J2 Pi_Zero_2W, J3 Molex 10, J4 Molex 10, Q1 2N7002H, Q10 2N7002H, Q11 2N7002H, Q12 2N7002H, Q13 2N7002H, Q14 2N7002H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

Commit message: 4 layers
Signed-off-by: Kolbjørn Austreng <kolbjorn.austreng@example.com>
Parts:
- added G***: LOGO, hotline:dickbutt, F.Cu at (170.5, 102.7)
- moved C13 11.3 mm to (97.3, 95.0)
- moved R2 5.86 mm to (136.4, 78.2)
- moved R1 5.84 mm to (130.6, 78.2)
- moved C11 5.74 mm to (97.8, 105.0)
- moved C12 5.74 mm to (97.1, 101.2)
- moved Q2 4.25 mm to (152.1, 128.7)
- moved Q3 4.25 mm to (152.1, 124.5)
- moved R24 4.25 mm to (155.3, 128.7)
- moved R25 4.25 mm to (155.3, 124.4)
- moved R26 4.25 mm to (157.8, 124.4)
- moved R27 4.25 mm to (157.8, 128.7)
- moved C19 2.01 mm to (110.6, 116.7)
- moved R19 2.01 mm to (110.6, 114.8)
- moved R13 1.57 mm to (170.7, 72.5)
- moved R39 1.57 mm to (168.7, 72.5)
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Connections:
- J2 pad 10: /LB -> /LE
- J2 pad 13: /BUTTON_R -> /LDP
- J2 pad 15: /LE -> /LB
- J2 pad 16: /LF -> /LC
- J2 pad 18: /LG -> /LA
- J2 pad 19: /RDP -> /RG
- J2 pad 21: /RG -> /RE
- J2 pad 22: /LDP -> /RF
- J2 pad 24: /RF -> /RD
- J2 pad 26: /RE -> /RDP
- J2 pad 3: /RA -> /BUTTON_L
- J2 pad 31: /RD -> /RB
- J2 pad 32: /Audio Out/AUDIO_L -> /Audio Out/AUDIO_R
- J2 pad 33: /Audio Out/AUDIO_R -> /Audio Out/AUDIO_L
- J2 pad 36: /LC -> /RA
- J2 pad 37: /BUTTON_L -> /BUTTON_R
- J2 pad 5: /RB -> /LF
- J2 pad 8: /LA -> /LG
Routing:
- net +3V3: track 0.00 -> 340.6 mm, vias 0 -> 15
- net GND: track 0.00 -> 96.1 mm, vias 0 -> 116
- net /Audio Out/AUDIO_R: track 0.00 -> 77.3 mm, vias 0 -> 1
- net /Audio Out/AUDIO_L: track 0.00 -> 72.7 mm, vias 0 -> 1
- net /BUTTON_L: track 0.00 -> 49.6 mm
- net /LG: track 0.00 -> 47.5 mm
- net /BUTTON_R: track 0.00 -> 45.1 mm
- net /RA: track 0.00 -> 44.6 mm
- net /LA: track 0.00 -> 44.5 mm
- net /RG: track 0.00 -> 41.1 mm
- net /RF: track 0.00 -> 39.6 mm
- net Net-(JP3-A): track 0.00 -> 38.0 mm
- net /RB: track 0.00 -> 37.9 mm
- net /LB: track 0.00 -> 37.4 mm
- net /LF: track 0.00 -> 37.3 mm
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- added copper zone on F.Cu, net +5V
- added copper zone on B.Cu, net GND
- added copper zone on In1.Cu, net GND
- added copper zone on In2.Cu, net GND
Other:
- board text added: "Hotline Dypet"
- board text added: "Kolbjørn Austreng"
- board text added: "v1"
