File: hotline/hotline.kicad_sch (KiCad schematic)
At the start: 32 parts, among them J1 Pi_Zero_2W, J2 USB_C_Receptacle_PowerOnly_24P, SW1 Left, SW2 Left, U1 PCM1808PWR, U2 LM4040DCK-2.0

Commit message: assign footprints
Signed-off-by: Kolbjørn Austreng <kolbjorn.austreng@example.com>
Parts:
- C1: renamed from C22; footprint (none) -> Capacitor_SMD:CP_Elec_6.3x7.7
- C10: renamed from C7; footprint (none) -> Capacitor_SMD:C_0603_1608Metric_Pad1.08x0.95mm_HandSolder
- C2: renamed from C3; footprint (none) -> Capacitor_SMD:CP_Elec_4x5.7
- C3: renamed from C5; footprint (none) -> Capacitor_SMD:CP_Elec_4x5.7
- C4: footprint (none) -> Capacitor_SMD:C_0603_1608Metric_Pad1.08x0.95mm_HandSolder
- C5: renamed from C6; footprint (none) -> Capacitor_SMD:C_0603_1608Metric_Pad1.08x0.95mm_HandSolder
- C6: renamed from C1; footprint (none) -> Capacitor_SMD:C_0603_1608Metric_Pad1.08x0.95mm_HandSolder
- C7: renamed from C21; footprint (none) -> Capacitor_SMD:C_0603_1608Metric_Pad1.08x0.95mm_HandSolder
- C8: renamed from C2; footprint (none) -> Capacitor_SMD:CP_Elec_4x5.7
- C9: renamed from C20; footprint (none) -> Capacitor_SMD:C_0603_1608Metric_Pad1.08x0.95mm_HandSolder
- D1: renamed from D3; footprint (none) -> Diode_SMD:D_0603_1608Metric_Pad1.05x0.95mm_HandSolder
- J1: renamed from J2; footprint (none) -> Connector_USB:USB_C_Receptacle_HRO_TYPE-C-31-M-17
- J2: renamed from J1; footprint (none) -> Connector_PinHeader_2.54mm:PinHeader_2x20_P2.54mm_Vertical
- MK1: footprint (none) -> TerminalBlock_Phoenix:TerminalBlock_Phoenix_PT-1,5-2-5.0-H_1x02_P5.00mm_Horizontal
- R1: renamed from R37; footprint (none) -> Resistor_SMD:R_0603_1608Metric_Pad0.98x0.95mm_HandSolder
- R10: renamed from R2; footprint (none) -> Resistor_SMD:R_0603_1608Metric_Pad0.98x0.95mm_HandSolder
- R11: renamed from R6; footprint (none) -> Resistor_SMD:R_0603_1608Metric_Pad0.98x0.95mm_HandSolder
- R12: renamed from R3; footprint (none) -> Resistor_SMD:R_0603_1608Metric_Pad0.98x0.95mm_HandSolder
- R13: renamed from R7; footprint (none) -> Resistor_SMD:R_0603_1608Metric_Pad0.98x0.95mm_HandSolder
- R2: renamed from R38; footprint (none) -> Resistor_SMD:R_0603_1608Metric_Pad0.98x0.95mm_HandSolder
- R3: renamed from R35; footprint (none) -> Resistor_SMD:R_0603_1608Metric_Pad0.98x0.95mm_HandSolder
- R4: renamed from R36; footprint (none) -> Resistor_SMD:R_0603_1608Metric_Pad0.98x0.95mm_HandSolder
- R5: renamed from R33; footprint (none) -> Resistor_SMD:R_0603_1608Metric_Pad0.98x0.95mm_HandSolder
- R6: renamed from R4; footprint (none) -> Resistor_SMD:R_0603_1608Metric_Pad0.98x0.95mm_HandSolder
- R7: renamed from R1; footprint (none) -> Resistor_SMD:R_0603_1608Metric_Pad0.98x0.95mm_HandSolder
- R8: renamed from R34; footprint (none) -> Resistor_SMD:R_0603_1608Metric_Pad0.98x0.95mm_HandSolder
- R9: renamed from R5; footprint (none) -> Resistor_SMD:R_0603_1608Metric_Pad0.98x0.95mm_HandSolder
- SW1: renamed from SW2; footprint (none) -> TerminalBlock_Phoenix:TerminalBlock_Phoenix_PT-1,5-2-5.0-H_1x02_P5.00mm_Horizontal
- SW2: renamed from SW1; value Left -> Right; footprint (none) -> TerminalBlock_Phoenix:TerminalBlock_Phoenix_PT-1,5-2-5.0-H_1x02_P5.00mm_Horizontal
- U1: footprint (none) -> Package_SO:TSSOP-14_4.4x5mm_P0.65mm
- renumbered D5 to D2

Commit message: place components
Signed-off-by: Kolbjørn Austreng <kolbjorn.austreng@example.com>
Parts:
- added H1, H2, H3, H4: MountingHole, symbol Mechanical:MountingHole
- added R39: 1k, Resistor_SMD:R_0603_1608Metric_Pad0.98x0.95mm_HandSolder, symbol Device:R_Small
Connections:
- net +3V3: now also R39.1; no longer R13.1, U2.3 (K)
- net at J1.B5 (CC2), R1.1: now also D2.2 (K); no longer D2.1 (K)
- net at J1.A5 (CC1), R2.1: now also D2.1 (K); no longer D2.2 (K)
- new net: R13.1, R39.2, U2.3 (K)
Other:
- moved on the sheet: U2

Commit message: 4 layers
Signed-off-by: Kolbjørn Austreng <kolbjorn.austreng@example.com>
Parts:
- H1, H2, H3, H4: footprint (none) -> MountingHole:MountingHole_2.2mm_M2_ISO7380_Pad
Connections:
- net Audio Out/AUDIO_L: now also J2.33 (PWM1/GPIO13); no longer J2.32 (PWM0/GPIO12)
- net Audio Out/AUDIO_R: now also J2.32 (PWM0/GPIO12); no longer J2.33 (PWM1/GPIO13)
- net BUTTON_L: now also J2.3 (SDA/GPIO2); no longer J2.37 (GPIO26)
- net BUTTON_R: now also J2.37 (GPIO26); no longer J2.13 (GPIO27)
- net LA: now also J2.18 (GPIO24); no longer J2.8 (GPIO14/TXD)
- net LB: now also J2.15 (GPIO22); no longer J2.10 (GPIO15/RXD)
- net LC: now also J2.16 (GPIO23); no longer J2.36 (GPIO16)
- net LDP: now also J2.13 (GPIO27); no longer J2.22 (GPIO25)
- net LE: now also J2.10 (GPIO15/RXD); no longer J2.15 (GPIO22)
- net LF: now also J2.5 (SCL/GPIO3); no longer J2.16 (GPIO23)
- net LG: now also J2.8 (GPIO14/TXD); no longer J2.18 (GPIO24)
- net RA: now also J2.36 (GPIO16); no longer J2.3 (SDA/GPIO2)
- net RB: now also J2.31 (GCLK2/GPIO6); no longer J2.5 (SCL/GPIO3)
- net RD: now also J2.24 (~{CE0}/GPIO8); no longer J2.31 (GCLK2/GPIO6)
- net RDP: now also J2.26 (~{CE1}/GPIO7); no longer J2.19 (MOSI0/GPIO10)
- net RE: now also J2.21 (MISO0/GPIO9); no longer J2.26 (~{CE1}/GPIO7)
- net RF: now also J2.22 (GPIO25); no longer J2.24 (~{CE0}/GPIO8)
- net RG: now also J2.19 (MOSI0/GPIO10); no longer J2.21 (MISO0/GPIO9)
Changed lines of the file:
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@@
 	)
 	(label "RDP"
-		(at 93.98 160.02 180)
+		(at 93.98 152.4 180)
 		(effects
 			(font
@@
 	)
 	(label "LE"
-		(at 24.13 154.94 0)
+		(at 24.13 129.54 0)
 		(effects
 			(font
@@
 	)
 	(label "LG"
-		(at 24.13 160.02 0)
+		(at 24.13 127 0)
 		(effects
 			(font
@@
 	)
 	(label "LDP"
-		(at 24.13 162.56 0)
+		(at 24.13 167.64 0)
 		(effects
 			(font
@@
 	)
 	(label "BUTTON_R"
-		(at 24.13 167.64 0)
+		(at 24.13 165.1 0)
 		(effects
 			(font
@@
 	)
 	(label "LA"
-		(at 24.13 127 0)
+		(at 24.13 160.02 0)
 		(effects
 			(font
@@
 	)
 	(label "BUTTON_L"
-		(at 24.13 165.1 0)
+		(at 93.98 134.62 180)
 		(effects
 			(font
 				(size 1.27 1.27)
 			)
-			(justify left bottom)
+			(justify right bottom)
 		)
 	)
@@
 	)
 	(label "RD"
-		(at 93.98 147.32 180)
+		(at 93.98 154.94 180)
 		(effects
 			(font
@@
 	)
 	(label "RE"
-		(at 93.98 152.4 180)
+		(at 93.98 157.48 180)
 		(effects
 			(font
@@
 	)
 	(label "RF"
-		(at 93.98 154.94 180)
+		(at 24.13 162.56 0)
 		(effects
 			(font
 				(size 1.27 1.27)
 			)
-			(justify right bottom)
+			(justify left bottom)
 		)
 	)
@@
 	)
 	(label "RG"
-		(at 93.98 157.48 180)
+		(at 93.98 160.02 180)
 		(effects
 			(font
@@
 	)
 	(label "LC"
-		(at 24.13 134.62 0)
+		(at 24.13 157.48 0)
 		(effects
 			(font
@@
 	)
 	(label "LB"
-		(at 24.13 129.54 0)
+		(at 24.13 154.94 0)
 		(effects
 			(font
@@
 	)
 	(label "LF"
-		(at 24.13 157.48 0)
+		(at 93.98 137.16 180)
 		(effects
 			(font
 				(size 1.27 1.27)
 			)
-			(justify left bottom)
+			(justify right bottom)
 		)
 	)
@@
 	)
 	(label "RA"
-		(at 93.98 134.62 180)
+		(at 24.13 134.62 0)
 		(effects
 			(font
 				(size 1.27 1.27)
 			)
-			(justify right bottom)
+			(justify left bottom)
 		)
 	)
 	(label "RB"
-		(at 93.98 137.16 180)
+		(at 93.98 147.32 180)
 		(effects
 			(font
@@
 			)
 		)
-		(property "Footprint" ""
+		(property "Footprint" "MountingHole:MountingHole_2.2mm_M2_ISO7380_Pad"
 			(at 248.92 100.33 0)
 			(effects
@@
 			)
 		)
-		(property "Footprint" ""
+		(property "Footprint" "MountingHole:MountingHole_2.2mm_M2_ISO7380_Pad"
 			(at 220.98 91.44 0)
 			(effects
@@
 			)
 		)
-		(property "Footprint" ""
+		(property "Footprint" "MountingHole:MountingHole_2.2mm_M2_ISO7380_Pad"
 			(at 220.98 100.33 0)
 			(effects
@@
 			)
 		)
-		(property "Footprint" ""
+		(property "Footprint" "MountingHole:MountingHole_2.2mm_M2_ISO7380_Pad"
 			(at 248.92 91.44 0)
 			(effects
@@
 		)
 		(pin "AUDIO_L" input
-			(at 105.41 167.64 180)
+			(at 105.41 170.18 180)
 			(effects
 				(font
@@
 		)
 		(pin "AUDIO_R" input
-			(at 105.41 170.18 180)
+			(at 105.41 167.64 180)
 			(effects
 				(font
